Commit message: 在虚拟机上尝试了双环PD，但是效果不好

File: BasicWBR/SlovedOnes/wbrtest_ws/src/wbrtestpkg/xacro/robotmodel.xacro (robot description, xacro)
@@ -4,5 +4,5 @@
      For more information, please see http://wiki.ros.org/sw_urdf_exporter -->
 <robot
-  name="wbrbodytest"  xmlns:xacro="http://wiki.ros.org/xacro">
+  name="wbrtestpkg"  xmlns:xacro="http://wiki.ros.org/xacro">
   <link
     name="base_link">
@@ -27,19 +27,19 @@
       <geometry>
         <mesh
-          filename="package://wbrbodytest/meshes/base_link.STL" />
-      </geometry>
-      <material
-        name="mt1">
-        <color
-          rgba="0.89804 0.91765 0.92941 1" />
-      </material>
-    </visual>
-    <collision>
-      <origin
-        xyz="0 0 0"
-        rpy="0 0 0" />
-      <geometry>
-        <mesh
-          filename="package://wbrbodytest/meshes/base_link.STL" />
+          filename="package://wbrtestpkg/meshes/base_link.STL" />
+      </geometry>
+      <material
+        name="mt1">
+        <color
+          rgba="0.89804 0.91765 0.92941 1" />
+      </material>
+    </visual>
+    <collision>
+      <origin
+        xyz="0 0 0"
+        rpy="0 0 0" />
+      <geometry>
+        <mesh
+          filename="package://wbrtestpkg/meshes/base_link.STL" />
       </geometry>
     </collision>
@@ -67,19 +67,19 @@
       <geometry>
         <mesh
-          filename="package://wbrbodytest/meshes/left_thigh.STL" />
-      </geometry>
-      <material
-        name="mt1">
-        <color
-          rgba="0.89804 0.91765 0.92941 1" />
-      </material>
-    </visual>
-    <collision>
-      <origin
-        xyz="0 0 0"
-        rpy="0 0 0" />
-      <geometry>
-        <mesh
-          filename="package://wbrbodytest/meshes/left_thigh.STL" />
+          filename="package://wbrtestpkg/meshes/left_thigh.STL" />
+      </geometry>
+      <material
+        name="mt1">
+        <color
+          rgba="0.89804 0.91765 0.92941 1" />
+      </material>
+    </visual>
+    <collision>
+      <origin
+        xyz="0 0 0"
+        rpy="0 0 0" />
+      <geometry>
+        <mesh
+          filename="package://wbrtestpkg/meshes/left_thigh.STL" />
       </geometry>
     </collision>
@@ -125,19 +125,19 @@
       <geometry>
         <mesh
-          filename="package://wbrbodytest/meshes/left_shank.STL" />
-      </geometry>
-      <material
-        name="mt1">
-        <color
-          rgba="0.89804 0.91765 0.92941 1" />
-      </material>
-    </visual>
-    <collision>
-      <origin
-        xyz="0 0 0"
-        rpy="0 0 0" />
-      <geometry>
-        <mesh
-          filename="package://wbrbodytest/meshes/left_shank.STL" />
+          filename="package://wbrtestpkg/meshes/left_shank.STL" />
+      </geometry>
+      <material
+        name="mt1">
+        <color
+          rgba="0.89804 0.91765 0.92941 1" />
+      </material>
+    </visual>
+    <collision>
+      <origin
+        xyz="0 0 0"
+        rpy="0 0 0" />
+      <geometry>
+        <mesh
+          filename="package://wbrtestpkg/meshes/left_shank.STL" />
       </geometry>
     </collision>
@@ -183,19 +183,19 @@
       <geometry>
         <mesh
-          filename="package://wbrbodytest/meshes/left_wheel.STL" />
-      </geometry>
-      <material
-        name="mt1">
-        <color
-          rgba="0.89804 0.91765 0.92941 1" />
-      </material>
-    </visual>
-    <collision>
-      <origin
-        xyz="0 0 0"
-        rpy="0 0 0" />
-      <geometry>
-        <mesh
-          filename="package://wbrbodytest/meshes/left_wheel.STL" />
+          filename="package://wbrtestpkg/meshes/left_wheel.STL" />
+      </geometry>
+      <material
+        name="mt1">
+        <color
+          rgba="0.89804 0.91765 0.92941 1" />
+      </material>
+    </visual>
+    <collision>
+      <origin
+        xyz="0 0 0"
+        rpy="0 0 0" />
+      <geometry>
+        <mesh
+          filename="package://wbrtestpkg/meshes/left_wheel.STL" />
       </geometry>
     </collision>
@@ -237,19 +237,19 @@
       <geometry>
         <mesh
-          filename="package://wbrbodytest/meshes/right_thigh.STL" />
-      </geometry>
-      <material
-        name="mt1">
-        <color
-          rgba="0.89804 0.91765 0.92941 1" />
-      </material>
-    </visual>
-    <collision>
-      <origin
-        xyz="0 0 0"
-        rpy="0 0 0" />
-      <geometry>
-        <mesh
-          filename="package://wbrbodytest/meshes/right_thigh.STL" />
+          filename="package://wbrtestpkg/meshes/right_thigh.STL" />
+      </geometry>
+      <material
+        name="mt1">
+        <color
+          rgba="0.89804 0.91765 0.92941 1" />
+      </material>
+    </visual>
+    <collision>
+      <origin
+        xyz="0 0 0"
+        rpy="0 0 0" />
+      <geometry>
+        <mesh
+          filename="package://wbrtestpkg/meshes/right_thigh.STL" />
       </geometry>
     </collision>
@@ -295,19 +295,19 @@
       <geometry>
         <mesh
-          filename="package://wbrbodytest/meshes/right_shank.STL" />
-      </geometry>
-      <material
-        name="mt1">
-        <color
-          rgba="0.89804 0.91765 0.92941 1" />
-      </material>
-    </visual>
-    <collision>
-      <origin
-        xyz="0 0 0"
-        rpy="0 0 0" />
-      <geometry>
-        <mesh
-          filename="package://wbrbodytest/meshes/right_shank.STL" />
+          filename="package://wbrtestpkg/meshes/right_shank.STL" />
+      </geometry>
+      <material
+        name="mt1">
+        <color
+          rgba="0.89804 0.91765 0.92941 1" />
+      </material>
+    </visual>
+    <collision>
+      <origin
+        xyz="0 0 0"
+        rpy="0 0 0" />
+      <geometry>
+        <mesh
+          filename="package://wbrtestpkg/meshes/right_shank.STL" />
       </geometry>
     </collision>
@@ -353,19 +353,19 @@
       <geometry>
         <mesh
-          filename="package://wbrbodytest/meshes/right_wheel.STL" />
-      </geometry>
-      <material
-        name="mt1">
-        <color
-          rgba="0.89804 0.91765 0.92941 1" />
-      </material>
-    </visual>
-    <collision>
-      <origin
-        xyz="0 0 0"
-        rpy="0 0 0" />
-      <geometry>
-        <mesh
-          filename="package://wbrbodytest/meshes/right_wheel.STL" />
+          filename="package://wbrtestpkg/meshes/right_wheel.STL" />
+      </geometry>
+      <material
+        name="mt1">
+        <color
+          rgba="0.89804 0.91765 0.92941 1" />
+      </material>
+    </visual>
+    <collision>
+      <origin
+        xyz="0 0 0"
+        rpy="0 0 0" />
+      <geometry>
+        <mesh
+          filename="package://wbrtestpkg/meshes/right_wheel.STL" />
       </geometry>
     </collision>
