Commit message: 跟换WBR2工程中的轮子为手动编写的urdf轮子，而非stl

File: WBR2_ws/src/wbr_pkg/xacro/actuators.xacro (robot description, xacro)
@@ -36,4 +36,5 @@
     <xacro:Effor_transmission_macro joint_name="Left_wheel_joint" />
     <!-- 使用位置控制的关节  -->
+    <!-- 这个joint_cond定义在robot.xacro 文件当中，用来判断是否使能关节位置控制 -->
     <xacro:if value = "${joint_cond}">
         <xacro:Position_transmission_macro joint_name="Right_knee_joint" />

File: WBR2_ws/src/wbr_pkg/xacro/robot_joint_fixed.xacro (robot description, xacro)
@@ -6,6 +6,9 @@
 <!-- 机器人的腿部关节全部指向左侧（z轴的正方向） -->
 <!-- 机器人完全站立的角度被定义为运动学的0位置  -->
-  <xacro:property name="hip_angle" value="0.7" />
-  <xacro:property name="knee_angle" value="-0.7" />
+  <!-- <xacro:property name="hip_angle" value="0.531" />
+  <xacro:property name="knee_angle" value="-0.923" /> -->
+1
+  <xacro:property name="hip_angle" value="0.367" />
+  <xacro:property name="knee_angle" value="-0.641" />
   <joint
     name="Left_hip_joint"

File: WBR2_ws/src/wbr_pkg/xacro/robot_links.xacro (robot description, xacro)
@@ -4,4 +4,5 @@
      For more information, please see http://wiki.ros.org/sw_urdf_exporter -->
 <robot name="robot_links" xmlns:xacro="http://wiki.ros.org/xacro">
+  <xacro:property name="is_stl_wheel" value="0" />
   <link name = "foot_print">
     <visual>
@@ -61,4 +62,8 @@
     </collision>
   </link>
+  <gazebo reference = "base_link">
+    <mu1>0.01</mu1>
+    <mu2>0.01</mu2>
+  </gazebo>
 <!-- *********************************************************************************************************************************** -->
   <link
@@ -144,4 +149,129 @@
   </link>
 <!-- *********************************************************************************************************************************** -->
+<!-- *********************************************************************************************************************************** -->
+  <link
+    name="Right_thigh_link">
+    <inertial>
+      <origin
+        xyz="0.1 0 -0.0175"
+        rpy="0 0 0" />
+      <mass
+        value="2.258" />
+      <inertia
+        ixx="0.0020663"
+        ixy="-5.2292E-20"
+        ixz="-6.4586E-21"
+        iyy="0.014683"
+        iyz="0"
+        izz="0.016288" />
+    </inertial>
+    <visual>
+      <origin
+        xyz="0 0 0"
+        rpy="0 0 0" />
+      <geometry>
+        <mesh
+          filename="package://wbr_pkg/meshes/Right_thigh_link.STL" />
+      </geometry>
+      <material
+        name="">
+        <color
+          rgba="1 1 1 1" />
+      </material>
+    </visual>
+    <collision>
+      <origin
+        xyz="0 0 0"
+        rpy="0 0 0" />
+      <geometry>
+        <mesh
+          filename="package://wbr_pkg/meshes/Right_thigh_link.STL" />
+      </geometry>
+    </collision>
+  </link>
+<!-- *********************************************************************************************************************************** -->
+  <link
+    name="Right_shank_link">
+    <inertial>
+      <origin
+        xyz="0.09 5.5511E-17 -0.0175"
+        rpy="0 0 0" />
+      <mass
+        value="2.0872" />
+      <inertia
+        ixx="0.0019065"
+        ixy="-7.382E-19"
+        ixz="-4.9947E-20"
+        iyy="0.011793"
+        iyz="-1.7781E-20"
+        izz="0.013273" />
+    </inertial>
+    <visual>
+      <origin
+        xyz="0 0 0"
+        rpy="0 0 0" />
+      <geometry>
+        <mesh
+          filename="package://wbr_pkg/meshes/Right_shank_link.STL" />
+      </geometry>
+      <material
+        name="">
+        <color
+          rgba="0.84706 0.84706 0.84706 1" />
+      </material>
+    </visual>
+    <collision>
+      <origin
+        xyz="0 0 0"
+        rpy="0 0 0" />
+      <geometry>
+        <mesh
+          filename="package://wbr_pkg/meshes/Right_shank_link.STL" />
+      </geometry>
+    </collision>
+  </link>
+<!-- *********************************************************************************************************************************** -->
+  <!-- 当 is_stl_wheel 为 true 的时候，将使用stl的轮子 -->
+  <xacro:if value = "${is_stl_wheel}">
+  <link
+    name="Right_wheel_link">
+    <inertial>
+      <origin
+        xyz="0 -2.7756E-17 -0.0175"
+        rpy="0 0 0" />
+      <mass
+        value="1.6567" />
+      <inertia
+        ixx="0.002913"
+        ixy="0"
+        ixz="4.8088E-36"
+        iyy="0.002913"
+        iyz="-7.283E-35"
+        izz="0.0054878" />
+    </inertial>
+    <visual>
+      <origin
+        xyz="0 0 0"
+        rpy="0 0 0" />
+      <geometry>
+        <mesh
+          filename="package://wbr_pkg/meshes/Right_wheel_link.STL" />
+      </geometry>
+      <material
+        name="">
+        <color
+          rgba="0.84706 0.84706 0.84706 1" />
+      </material>
+    </visual>
+    <collision>
+      <origin
+        xyz="0 0 0"
+        rpy="0 0 0" />
+      <geometry>
+        <mesh
+          filename="package://wbr_pkg/meshes/Right_wheel_link.STL" />
+      </geometry>
+    </collision>
+  </link>
   <link
     name="Left_wheel_link">
@@ -184,126 +314,81 @@
     </collision>
   </link>
-<!-- *********************************************************************************************************************************** -->
-  <link
-    name="Right_thigh_link">
-    <inertial>
-      <origin
-        xyz="0.1 0 -0.0175"
-        rpy="0 0 0" />
-      <mass
-        value="2.258" />
-      <inertia
-        ixx="0.0020663"
-        ixy="-5.2292E-20"
-        ixz="-6.4586E-21"
-        iyy="0.014683"
-        iyz="0"
-        izz="0.016288" />
-    </inertial>
-    <visual>
-      <origin
-        xyz="0 0 0"
-        rpy="0 0 0" />
-      <geometry>
-        <mesh
-          filename="package://wbr_pkg/meshes/Right_thigh_link.STL" />
-      </geometry>
-      <material
-        name="">
-        <color
-          rgba="1 1 1 1" />
-      </material>
-    </visual>
-    <collision>
-      <origin
-        xyz="0 0 0"
-        rpy="0 0 0" />
-      <geometry>
-        <mesh
-          filename="package://wbr_pkg/meshes/Right_thigh_link.STL" />
-      </geometry>
-    </collision>
-  </link>
-<!-- *********************************************************************************************************************************** -->
-  <link
-    name="Right_shank_link">
-    <inertial>
-      <origin
-        xyz="0.09 5.5511E-17 -0.0175"
-        rpy="0 0 0" />
-      <mass
-        value="2.0872" />
-      <inertia
-        ixx="0.0019065"
-        ixy="-7.382E-19"
-        ixz="-4.9947E-20"
-        iyy="0.011793"
-        iyz="-1.7781E-20"
-        izz="0.013273" />
-    </inertial>
-    <visual>
-      <origin
-        xyz="0 0 0"
-        rpy="0 0 0" />
-      <geometry>
-        <mesh
-          filename="package://wbr_pkg/meshes/Right_shank_link.STL" />
-      </geometry>
-      <material
-        name="">
-        <color
-          rgba="0.84706 0.84706 0.84706 1" />
-      </material>
-    </visual>
-    <collision>
-      <origin
-        xyz="0 0 0"
-        rpy="0 0 0" />
-      <geometry>
-        <mesh
-          filename="package://wbr_pkg/meshes/Right_shank_link.STL" />
-      </geometry>
-    </collision>
-  </link>
-<!-- *********************************************************************************************************************************** -->
+  </xacro:if>
+  <!-- 当 is_stl_wheel 为 false 的时候，将使用下方urdf直接建模的轮子 -->
+  <xacro:property name = "wheel_r" value = "0.08"/>
+  <xacro:property name = "wheel_h" value = "0.035"/>
+  <xacro:property name = "wheel_m" value = "1.6567"/>
+  <xacro:macro name="cylinder_inertial_matrix" params="m r h">
+    <!-- <inertial>
+      <origin
+        xyz="0 0 0.0175"
+        rpy="0 0 0" /> -->
+      <mass value="${m}" />
+      <inertia ixx="${m*(3*r*r+h*h)/12}" ixy = "0" ixz = "0"
+        iyy="${m*(3*r*r+h*h)/12}" iyz = "0"
+        izz="${m*r*r/2}" />
+    <!-- </inertial> -->
+  </xacro:macro>
+  <xacro:unless value = "${is_stl_wheel}">
   <link
     name="Right_wheel_link">
     <inertial>
       <origin
-        xyz="0 -2.7756E-17 -0.0175"
-        rpy="0 0 0" />
-      <mass
-        value="1.6567" />
-      <inertia
-        ixx="0.002913"
-        ixy="0"
-        ixz="4.8088E-36"
-        iyy="0.002913"
-        iyz="-7.283E-35"
-        izz="0.0054878" />
-    </inertial>
-    <visual>
-      <origin
-        xyz="0 0 0"
-        rpy="0 0 0" />
-      <geometry>
-        <mesh
-          filename="package://wbr_pkg/meshes/Right_wheel_link.STL" />
-      </geometry>
-      <material
-        name="">
-        <color
-          rgba="0.84706 0.84706 0.84706 1" />
-      </material>
-    </visual>
-    <collision>
-      <origin
-        xyz="0 0 0"
-        rpy="0 0 0" />
-      <geometry>
-        <mesh
-          filename="package://wbr_pkg/meshes/Right_wheel_link.STL" />
-      </geometry>
-    </collision>
-  </link>
+        xyz="0 0 -0.0175"
+        rpy="0 0 0" />
+      <xacro:cylinder_inertial_matrix m="${wheel_m}" r="${wheel_r}" h="${wheel_h}" />
+    </inertial>
+    <visual>
+      <origin
+        xyz="0 0 -0.0175"
+        rpy="0 0 0" />
+      <geometry>
+          <cylinder radius="${wheel_r}" length="${wheel_h}"/>
+      </geometry>
+      <material
+        name="">
+        <color
+          rgba="0.84706 0.84706 0.84706 1" />
+      </material>
+    </visual>
+    <collision>
+      <origin
+        xyz="0 0 -0.0175"
+        rpy="0 0 0" />
+      <geometry>
+         <cylinder radius="${wheel_r}" length="${wheel_h}"/>
+      </geometry>
+    </collision>
+  </link>
+  <link
+    name="Left_wheel_link">
+    <inertial>
+      <origin
+        xyz="0 0 0.0175"
+        rpy="0 0 0" />
+      <xacro:cylinder_inertial_matrix m="${wheel_m}" r="${wheel_r}" h="${wheel_h}" />
+    </inertial>
+    <visual>
+      <origin
+        xyz="0 0 0.0175"
+        rpy="0 0 0" />
+      <geometry>
+          <cylinder radius="${wheel_r}" length="${wheel_h}"/>
+      </geometry>
+      <material
+        name="">
+        <color
+          rgba="0.84706 0.84706 0.84706 1" />
+      </material>
+    </visual>
+    <collision>
+      <origin
+        xyz="0 0 0.0175"
+        rpy="0 0 0" />
+      <geometry>
+         <cylinder radius="${wheel_r}" length="${wheel_h}"/>
+      </geometry>
+    </collision>
+  </link>
+  </xacro:unless>
 </robot>

Commit message: WBR2的整个工程文件应该来说是完成了，缺点就是LQR不好使

File: WBR2_ws/src/wbr_pkg/xacro/actuators.xacro (robot description, xacro)
@@ -37,5 +37,5 @@
     <!-- 使用位置控制的关节  -->
     <!-- 这个joint_cond定义在robot.xacro 文件当中，用来判断是否使能关节位置控制 -->
-    <xacro:if value = "${joint_cond}">
+    <xacro:if value = "${is_joint_movable}">
         <xacro:Position_transmission_macro joint_name="Right_knee_joint" />
         <xacro:Position_transmission_macro joint_name="Right_hip_joint" />

File: WBR2_ws/src/wbr_pkg/xacro/robot.xacro (robot description, xacro)
@@ -2,13 +2,13 @@
     <xacro:include filename="robot_links.xacro" />
     <!-- 调用机器人模型 -->
-    <xacro:property name="joint_cond" value="0" />
-    <!-- 1:允许关节运动 0 ：关节锁死 -->
+    <xacro:property name="is_joint_movable" value="0" />
+    <!-- 1:允许关节运动 0 ：关节锁死; 另外，可能需要修改yaml文件... -->
     <!-- 0:不允许关节运动，即关节锁死 -->
-    <xacro:unless value= "${joint_cond}">
+    <xacro:unless value= "${is_joint_movable}">
         <xacro:include filename="robot_joint_fixed.xacro" />
         <!-- 关节锁死（可以在此文件中修改关节偏置量）-->
     </xacro:unless>
     <!-- 1: 允许关节运动，可以启动关节位置控制甚至力控制器 -->
-    <xacro:if value = "${joint_cond}">
+    <xacro:if value = "${is_joint_movable}">
         <xacro:include filename="robot_joint_revolute.xacro" />
     </xacro:if>
