Commit message: 为了实现RMer设计的模型，设计了一个urdf文件，但是在octave推导中发现，论文的系统根本就是不稳定的（恼）

File: BasicLQR/basicwip_ws/src/rmer_lqr_pkg/xacro/robotmodel.xacro (robot description, xacro)
@@ -27,5 +27,5 @@
       <visual>
         <geometry>
-          <box size="0.01 0.5 0.01"/>
+          <box size="0.02 0.5 0.02"/>
         </geometry>
         <origin xyz="0 0 0" rpy="0 0 0" />
@@ -36,9 +36,11 @@
       <collision>
         <geometry>
-          <box size="0.01 0.5 0.01"/>
+          <box size="0.02 0.5 0.02"/>
         </geometry>
         <origin xyz="0 0 0" rpy="0 0 0" />
       </collision>
-      <xacro:Box_inertial_matrix m="0.01" w="0.01" h="0.5" l = "0.01" />
+      <inertial>
+        <xacro:Box_inertial_matrix m="0.01" w="0.02" h="0.5" l = "0.02" />
+      </inertial>
     </link>
     <joint name="base_link2base_footprint" type="fixed">
@@ -53,5 +55,5 @@
       <visual>
         <geometry>
-         <box size="0.01 0.01 0.5"/>
+         <box size="0.02 0.02 0.5"/>
         </geometry>
         <origin xyz="0 0 0" rpy="0 0 0" />
@@ -62,12 +64,12 @@
       <collision>
         <geometry>
-          <box size="0.01 0.01 0.5"/>
+          <box size="0.02 0.02 0.5"/>
         </geometry>
         <origin xyz="0 0 0" rpy="0 0 0" />
       </collision>
-      <inertia>
+      <inertial>
         <!-- 这里给了杆一个质量，为了控制的时候考虑这部分内容。 -->
-        <xacro:Box_inertial_matrix m="0.5" w="0.01" h="0.01" l = "0.5" />
-      </inertia>
+        <xacro:Box_inertial_matrix m="0.5" w="0.02" h="0.02" l = "0.5" />
+      </inertial>
     </link>
     <joint name="base2vertial_link" type="fixed">
@@ -112,5 +114,5 @@
       <visual>
         <geometry>
-         <sphere radius = "0.1"/>
+         <box size="0.3 0.3 0.2"/>
         </geometry>
         <origin xyz="0 0 0" rpy="0 0 0" />
@@ -121,14 +123,18 @@
       <collision>
         <geometry>
-          <sphere radius = "0.1"/>
+          <box size="0.3 0.3 0.2"/>
         </geometry>
         <origin xyz="0 0 0" rpy="0 0 0" />
       </collision>
-      <xacro:sphere_inertial_matrix m="10" r="0.1" />
+      <inertial>
+        <xacro:Box_inertial_matrix m="10" w="0.3" h="0.3" l = "0.2" />
+      </inertial>
     </link>
-    <joint name="mass2vertial_joint" type="fixed">
+    <joint name="mass2vertial_joint" type="revolute">
       <parent link="vertical_link" />
       <child link="mass_link" />
       <origin xyz="0 0 0.25" />
+      <axis xyz = "0 1 0"/>
+      <limit lower="-1.57" upper="1.57" effort="50" velocity="20.0"/>
     </joint>
     <gazebo reference="mass_link">
